Commit message: GripX Orientation

File: gripx_description/urdf/gripx_gazebo.urdf (robot description, URDF)
Before this commit: robot gripx, 8 links, 7 joints
Joints:
- joint joint_6: limit lower=-2.57 upper=2.57 effort=7 velocity=1.6 -> lower=-3.57 upper=3.57 effort=7 velocity=1.6; origin xyz=-0.45 0 0.01872799 rpy=0 0 0 -> xyz=-0.485 0.0 0.03 rpy=0 0 0
